File: KiCad-9/MusicalTeslaCoil.kicad_pcb (KiCad board)
At the start: 4 copper layers, 100 x 100 mm, 117 parts, among them J1 USB_C-UJ20-C-H-C-MSMT-TR, J10 NTC Thermistor 2, J11 Conn_01x10_Pin, J12 Conn_01x05_Pin, J13 Conn_01x06_Pin, J14 Conn_02x03_Odd_Even, J2 Power in, J3 VBUS, J4 Primary Relay, J5 Soft Start Bypass Relay, J6 Current Transformer, J7 GDT1, J8 GDT2, J9 NTC Thermistor 1, Q1 PMV20ENR, Q2 PMV20ENR, SW1 USB Boot, SW2 Reset, U1 ESP32-S3-WROOM-1, U10 AP2112K-3.3TRG1, U2 R1240N001B-TR-FE, U3 LMV321, U4 DMC4029SK4-13, U5 UCC27423DR, U6 DMC4029SK4-13, U7 UCC27423DR, U8 DMC4029SK4-13, U9 DMC4029SK4-13

Commit message: Uploaded Rev 2.0
Parts:
- removed the C36 at (65.5, 55.9)
- removed the C37 at (65.5, 62.8)
- removed the C38 at (90.7, 127.2)
- removed the C39 at (81.0, 128.9)
- removed the C40 at (65.6, 147.0)
- removed the C41 at (74.5, 129.0)
- removed the CR12 at (62.5, 90.8)
- removed the CR13 at (67.4, 137.5)
- removed the J1 at (50.8, 87.2)
- removed the R34 at (77.5, 138.0)
- removed the R35 at (77.0, 129.0)
- removed the R36 at (77.0, 133.5)
- removed the U10 at (86.8, 127.0)
- added C13: 10nF, Capacitor_SMD:C_0805_2012Metric_Pad1.18x1.45mm_HandSolder, F.Cu at (102.0, 88.5)
- added C14: 0.1uF, Capacitor_SMD:C_0805_2012Metric_Pad1.18x1.45mm_HandSolder, F.Cu at (79.0, 143.0)
- added C15: 10nF, Capacitor_SMD:C_0805_2012Metric_Pad1.18x1.45mm_HandSolder, F.Cu at (102.0, 85.0)
- added C16: 10nF, Capacitor_SMD:C_0805_2012Metric_Pad1.18x1.45mm_HandSolder, F.Cu at (91.1, 143.6)
- added C17: 10uF, Capacitor_SMD:C_0805_2012Metric_Pad1.18x1.45mm_HandSolder, F.Cu at (68.4, 128.6)
- added C18: 2.2uF, Capacitor_SMD:C_0805_2012Metric_Pad1.18x1.45mm_HandSolder, F.Cu at (94.5, 142.6)
- added C19: 10uF, Capacitor_SMD:C_0805_2012Metric_Pad1.18x1.45mm_HandSolder, F.Cu at (66.0, 128.6)
- added C2: 10uF, Capacitor_SMD:C_0805_2012Metric_Pad1.18x1.45mm_HandSolder, F.Cu at (70.4, 138.7)
- added C20: 2.2uF, Capacitor_SMD:C_0805_2012Metric_Pad1.18x1.45mm_HandSolder, F.Cu at (111.5, 84.5)
- added C21: 1nF, Capacitor_SMD:C_0805_2012Metric_Pad1.18x1.45mm_HandSolder, F.Cu at (114.5, 89.5)
- added C22: 2.2uF, Capacitor_SMD:C_0805_2012Metric_Pad1.18x1.45mm_HandSolder, F.Cu at (117.5, 94.0)
- added C29: 2.2uF, Capacitor_SMD:C_0805_2012Metric_Pad1.18x1.45mm_HandSolder, F.Cu at (120.9, 93.0)
- added C3: 2.2uF, Capacitor_SMD:C_0805_2012Metric_Pad1.18x1.45mm_HandSolder, F.Cu at (54.9, 129.1)
- added C4: 10nF, Capacitor_SMD:C_0805_2012Metric_Pad1.18x1.45mm_HandSolder, F.Cu at (102.0, 95.5)
- added C45: 1uF, Capacitor_SMD:C_0805_2012Metric_Pad1.18x1.45mm_HandSolder, F.Cu at (93.4, 98.6)
- added C46: 1uF, Capacitor_SMD:C_0805_2012Metric_Pad1.18x1.45mm_HandSolder, F.Cu at (84.9, 86.3)
- added C53: 470pF, Capacitor_SMD:C_0805_2012Metric_Pad1.18x1.45mm_HandSolder, F.Cu at (77.9, 90.2)
- added C6: 1uF, Capacitor_SMD:C_0805_2012Metric_Pad1.18x1.45mm_HandSolder, F.Cu at (87.4, 86.3)
- added CR1: MSS1P4-M3/89A, MSS1P4_M3_89A:DIODE_MSP3V3, F.Cu at (60.6, 88.9)
- added CR10: MSS1P4-M3/89A, MSS1P4_M3_89A:DIODE_MSP3V3, F.Cu at (93.5, 105.0)
- added CR9: MSS1P4-M3/89A, MSS1P4_M3_89A:DIODE_MSP3V3, F.Cu at (87.0, 103.3)
- added D9: BZT52C15-7-F, Diode_SMD:D_SOD-123, F.Cu at (64.7, 149.3)
- added F1: 0ZCG0050AF2C, 0ZCG0050AF2C:FUSER_0ZCG0050AF2C, F.Cu at (65.6, 144.2)
- added H1: MountingHole, MountingHole:MountingHole_3.2mm_M3, F.Cu at (144.4, 57.1)
- added H2: MountingHole, MountingHole:MountingHole_3.2mm_M3, F.Cu at (53.6, 57.1)
- added H3: MountingHole, MountingHole:MountingHole_3.2mm_M3, F.Cu at (144.4, 147.9)
- added H4: MountingHole, MountingHole:MountingHole_3.2mm_M3, F.Cu at (53.6, 147.9)
- added J17: Conn_01x05, Connector_PinHeader_2.54mm:PinHeader_1x05_P2.54mm_Vertical, F.Cu at (83.6, 66.5)
- added J18: Conn_01x07, Connector_PinHeader_2.54mm:PinHeader_1x07_P2.54mm_Vertical, F.Cu at (121.9, 55.5)
- added J2: Conn_01x03, Connector_Molex:Molex_KK-254_AE-6410-03A_1x03_P2.54mm_Vertical, F.Cu at (94.4, 77.6)
- added J3: USB4215-03-A, USB4215_03_A:USB4215_03_A, F.Cu at (51.4, 85.5)
- added LED1: LTST-C170GKT, LTST_C170GKT:LED_LTST-C170GKT_LTO, F.Cu at (57.1, 121.0)
- added LED2: LTST-C170KFKT, LTST_C170KFKT:LED_LTST-C170KFKT_LTO, F.Cu at (80.5, 78.9)
- added LED3: LTST-C171KRKT, LTST_C171KRKT:LED_LTST-C171_LTO, F.Cu at (71.5, 78.9)
- added LED4: LTST-C170KSKT, LTST_C170KSKT:LED_LTST-C170KSKT_LTO, F.Cu at (85.0, 79.0)
- added LED5: LTST-C170GKT, LTST_C170GKT:LED_LTST-C170GKT_LTO, F.Cu at (76.0, 79.1)
- added Q5: 2N7002K, Package_TO_SOT_SMD:SOT-23, F.Cu at (136.0, 75.0)
- added Q6: 2N7002K, Package_TO_SOT_SMD:SOT-23, F.Cu at (135.9, 87.5)
- added R1: 5.1k, Resistor_SMD:R_0805_2012Metric_Pad1.20x1.40mm_HandSolder, F.Cu at (69.7, 149.3)
- added R10: 100k, Resistor_SMD:R_0805_2012Metric_Pad1.20x1.40mm_HandSolder, F.Cu at (54.6, 91.8)
- added R12: 1k, Resistor_SMD:R_0805_2012Metric_Pad1.20x1.40mm_HandSolder, F.Cu at (97.5, 92.0)
- added R14: 150, Resistor_SMD:R_0805_2012Metric_Pad1.20x1.40mm_HandSolder, F.Cu at (80.5, 74.5)
- added R15: 150, Resistor_SMD:R_0805_2012Metric_Pad1.20x1.40mm_HandSolder, F.Cu at (71.5, 74.5)
- added R16: 0, Resistor_SMD:R_0805_2012Metric_Pad1.20x1.40mm_HandSolder, F.Cu at (79.0, 139.0)
- added R17: 1k, Resistor_SMD:R_0805_2012Metric_Pad1.20x1.40mm_HandSolder, F.Cu at (97.5, 85.0)
- added R18: 5.1k, Resistor_SMD:R_0805_2012Metric_Pad1.20x1.40mm_HandSolder, F.Cu at (63.0, 88.8)
- added R19: 3k, Resistor_SMD:R_0805_2012Metric_Pad1.20x1.40mm_HandSolder, F.Cu at (91.0, 147.6)
- added R2: 3k, Resistor_SMD:R_0805_2012Metric_Pad1.20x1.40mm_HandSolder, F.Cu at (51.3, 129.1)
- added R20: 16.5k, Resistor_SMD:R_0805_2012Metric_Pad1.20x1.40mm_HandSolder, F.Cu at (86.5, 147.6)
- added R21: 150, Resistor_SMD:R_0805_2012Metric_Pad1.20x1.40mm_HandSolder, F.Cu at (85.0, 74.5)
- added R22: 150, Resistor_SMD:R_0805_2012Metric_Pad1.20x1.40mm_HandSolder, F.Cu at (76.0, 74.5)
- added R23: 22k, Resistor_SMD:R_0805_2012Metric_Pad1.20x1.40mm_HandSolder, F.Cu at (83.0, 139.0)
- added R24: 3k, Resistor_SMD:R_0805_2012Metric_Pad1.20x1.40mm_HandSolder, F.Cu at (83.0, 143.0)
- added R25: 10k, Resistor_SMD:R_0805_2012Metric_Pad1.20x1.40mm_HandSolder, F.Cu at (76.6, 124.2)
- added R26: 51, Resistor_SMD:R_0805_2012Metric_Pad1.20x1.40mm_HandSolder, F.Cu at (117.5, 89.5)
- added R29: 3k, Resistor_SMD:R_0805_2012Metric_Pad1.20x1.40mm_HandSolder, F.Cu at (129.5, 63.5)
- added R57: 150, Resistor_SMD:R_0805_2012Metric_Pad1.20x1.40mm_HandSolder, F.Cu at (77.9, 94.2)
- added R58: 200k, Resistor_SMD:R_0805_2012Metric_Pad1.20x1.40mm_HandSolder, F.Cu at (80.4, 90.2)
- added R6: 5.1k, Resistor_SMD:R_0805_2012Metric_Pad1.20x1.40mm_HandSolder, F.Cu at (63.0, 83.2)
- added U1: TLV75801PDBV, Package_TO_SOT_SMD:SOT-23-5, F.Cu at (58.8, 129.2)
- added U15: NCS2250SQ2T2G, NCS2250SQ2T2G:SC70-5_2P2X1P35_ONS, F.Cu at (90.4, 100.6)
- added U16: NCS2250SQ2T2G, NCS2250SQ2T2G:SC70-5_2P2X1P35_ONS, F.Cu at (83.9, 90.2)
- added U4: MCP3204T-CI/SL, MCP3204T_CI_SL:SOIC14-N_MC_MCH, F.Cu at (108.9, 91.2)
- added U5: MCP48FVB11, MCP48FVB11:MCP48FVB11, F.Cu at (90.0, 90.3)
- added U6: MCP1501T-33E/CHY, MCP1501T_33E_CHY:SOT-23-6_CHY_MCH, F.Cu at (121.7, 89.5)
- added U7: MCP6006UT-E/LT, MCP6006UT_E_LT:SC70-5_LT_MCH, F.Cu at (129.5, 68.9)
- C1: value 0.1uF -> 2.2uF
- C26: renamed from C42; value 1uF -> 0.1uF
- C5: value 10uF -> 2.2uF
- C7: value 1nF -> 10nF
- CR11: renamed from CR8; value 1N4007FL -> 1N4148WS-7-F; footprint 1N4007FL:CR_SOD-123FL_SME -> 1N4148WX_TP:CR_SOD323_MCC
- CR12: renamed from CR9; value 1N4007FL -> 1N4148WS-7-F; footprint 1N4007FL:CR_SOD-123FL_SME -> 1N4148WX_TP:CR_SOD323_MCC
- CR13: renamed from CR10; value 1N4007FL -> 1N4148WS-7-F; footprint 1N4007FL:CR_SOD-123FL_SME -> 1N4148WX_TP:CR_SOD323_MCC
- CR14: renamed from CR11; value 1N4007FL -> 1N4148WS-7-F; footprint 1N4007FL:CR_SOD-123FL_SME -> 1N4148WX_TP:CR_SOD323_MCC
- J11: value Conn_01x10_Pin -> Conn_01x02; footprint Connector_PinHeader_2.54mm:PinHeader_1x10_P2.54mm_Vertical -> Connector_Molex:Molex_KK-254_AE-6410-02A_1x02_P2.54mm_Vertical
- J12: value Conn_01x05_Pin -> Conn_01x02; footprint Connector_PinHeader_2.54mm:PinHeader_1x05_P2.54mm_Vertical -> Connector_Molex:Molex_KK-254_AE-6410-02A_1x02_P2.54mm_Vertical
- J13: value Conn_01x06_Pin -> Conn_01x02; footprint Connector_PinHeader_2.54mm:PinHeader_1x06_P2.54mm_Vertical -> Connector_Molex:Molex_KK-254_AE-6410-02A_1x02_P2.54mm_Vertical
- J14: value Conn_02x03_Odd_Even -> Conn_01x02; footprint Connector_PinHeader_2.54mm:PinHeader_2x03_P2.54mm_Vertical -> Connector_Molex:Molex_KK-254_AE-6410-02A_1x02_P2.54mm_Vertical
- L1: value SLF7045T-4R7M2R0-PF -> VLS6045EX-150M; footprint SLF7045T_4R7M2R0_PF:IND_7045_TDK -> VLS6045EX_150M:VLS6045EX_150M
- Q1: value PMV20ENR -> GSF3407; footprint PMV20ENR:QNMOS1G2S3D_TO-236AB_SOT23_NEX -> Package_TO_SOT_SMD:SOT-23
- Q2: value PMV20ENR -> SSF7912; footprint PMV20ENR:QNMOS1G2S3D_TO-236AB_SOT23_NEX -> Package_TO_SOT_SMD:SOT-23
- R11: value 5.1k -> 1k
- R27: renamed from R10; value 3k 1% -> 1.5k
- R3: value 5.1k -> 15k
- R31: renamed from R12; value 3k 1% -> 3k
- R33: renamed from R14; value 1k -> 10k
- R34: renamed from R17; value 1k -> 10k
- R35: renamed from R15; value 50 -> 51
- R36: renamed from R16; value 50 -> 51
- R37: renamed from R32; value 1k 1% -> 1k
- R38: renamed from R33; value 1k 1% -> 1k
- R51: renamed from R18; value 100 -> 1k
- R52: renamed from R19; value 100 -> 1k
- R7: value 100k -> 150
- U2: value R1240N001B-TR-FE -> TPP362082-T6TR; footprint R1240N001B_TR_FE:SOT-23-6W_PE-SOT23-6W-0512_NMD -> TPP362082_T6TR:TSOT23-6-A_TPK
- U3: value LMV321 -> TLV75801PDBV; footprint footprints:DCK5_TEX -> Package_TO_SOT_SMD:SOT-23-5
- moved Q1 106.7 mm to (59.5, 150.0), turned to 180 degrees
- moved U3 82.6 mm to (91.0, 139.6), turned to -90 degrees
- moved J11 70.0 mm to (89.6, 118.4), turned to 180 degrees
- moved Q2 68.1 mm to (80.5, 127.0), turned to 0 degrees
- moved J12 53.6 mm to (96.6, 118.4), turned to 180 degrees
- moved R11 39.2 mm to (97.5, 95.5), turned to 180 degrees
- moved R3 37.1 mm to (51.3, 125.1), turned to -90 degrees
- moved J13 36.1 mm to (103.8, 118.4), turned to 180 degrees
- moved R13 35.4 mm to (97.5, 88.5), turned to 180 degrees
- moved C7 33.3 mm to (102.0, 92.0), turned to 0 degrees
- moved R7 29.5 mm to (52.5, 121.0), turned to 180 degrees
- moved J14 23.4 mm to (111.0, 118.4), turned to 180 degrees
- moved C5 21.7 mm to (91.1, 135.6), turned to 180 degrees
- moved C33 21.0 mm to (72.7, 89.3), turned to 180 degrees
- moved R47 20.5 mm to (68.5, 93.0)
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- renumbered C6 to C23, C4 to C24, C2 to C25, C43 to C27, C3 to C28, C14 to C30, C15 to C31, C13 to C32, C17 to C33, C18 to C34, C27 to C35, C16 to C36, C19 to C37, C24 to C38, C28 to C39, C29 to C40, C20 to C41, C25 to C42, C30 to C43, C31 to C44, C21 to C47, C26 to C48, C32 to C49, C33 to C50, C22 to C51, C34 to C52, C23 to C54, C35 to C55, CR1 to CR2, CR2 to CR3, CR7 to CR4, CR4 to CR5, CR3 to CR6, CR6 to CR7, CR5 to CR8, J2 to J1, J5 to J10, J7 to J15, J8 to J16, J3 to J4, J6 to J5, J9 to J6, J10 to J7, J4 to J9, R6 to R28, R1 to R30, R2 to R32, R23 to R39, R27 to R43, R22 to R44, R28 to R45, R21 to R46, R20 to R47, R38 to R48, R37 to R49, R39 to R50, R24 to R53, R26 to R54, R29 to R55, R30 to R56, R25 to R59, R31 to R60, U7 to U10, U4 to U11, U6 to U12, U8 to U13, U9 to U14, U1 to U8, U5 to U9
Connections:
- C1 pad 1: Net-(U2-LX) -> GND
- C1 pad 2: Net-(C1-Pad2) -> 5V
- C23 pad 2: Net-(J3-Pin_2) -> Net-(J4-Pin_2)
- C26 pad 2: 3.3V -> A3.6V
- C27 pad 2: 3.3V -> D3.3V
- C28 pad 1: 3.3V -> D3.3V
- C33 pad 2: CTout -> CTOut
- C36 pad 1: ZCDB -> Net-(U15--)
- C36 pad 2: ZCDA -> Net-(U15-+)
- C5 pad 1: 24V -> GND
- C5 pad 2: GND -> 5V
- C7 pad 2: VBUS -> Net-(U4-CH2)
- CR2 pad 2: Net-(J4-Pin_2) -> Net-(J9-Pin_2)
- CR3 pad 2: Net-(J5-Pin_2) (its old number) -> Net-(J10-Pin_2)
- J1 pad 2: 24V -> Net-(J1-Pin_2)
- J10 pad 2: Net-(J5-Pin_2) (its old number) -> Net-(J10-Pin_2)
- J11 pad 1: TXD0 -> 24V
- J11 pad 2: RXD0 -> GND
- J12 pad 1: IO7 -> 5V
- J12 pad 2: IO15 -> GND
- J13 pad 1: IO9 -> A3.6V
- J13 pad 2: IO10 -> GND
- J14 pad 1: 5V -> D3.3V
- J4 pad 1: Net-(J3-Pin_1) -> Net-(J4-Pin_1)
- J4 pad 2: Net-(J3-Pin_2) -> Net-(J4-Pin_2)
- J6 pad 2: 3.3V -> A3.6V
- J7 pad 2: 3.3V -> A3.6V
- J9 pad 2: Net-(J4-Pin_2) -> Net-(J9-Pin_2)
- L1 pad 1: 5V -> Net-(U2-SW)
- L1 pad 2: Net-(U2-LX) -> Net-(Q2-S)
- Q1 pad 1: Net-(Q1-G) -> Net-(D9-A)
- Q1 pad 2: GND -> Net-(D9-K)
- Q1 pad 3: Net-(J4-Pin_2) -> Net-(J1-Pin_2)
- Q2 pad 1: Net-(Q2-G) -> 24V
- Q2 pad 2: GND -> Net-(Q2-S)
- Q2 pad 3: Net-(J5-Pin_2) (its old number) -> 5V
- R11 pad 1: GND -> Net-(U4-CH3)
- R13 pad 1: VBUS -> Net-(U4-CH1)
- R13 pad 2: Net-(R12-Pad1) -> Therm1
- R27 pad 2: Net-(J3-Pin_2) -> Net-(J4-Pin_2)
- R28 pad 1: 3.3V -> D3.3V
- R30 pad 1: 3.3V -> D3.3V
- R31 pad 1: Net-(R12-Pad1) -> VBUS
- R31 pad 2: Net-(J3-Pin_1) -> Net-(J4-Pin_1)
- R33 pad 1: Net-(Q1-G) -> PrimaryRelay
- R34 pad 1: Net-(Q2-G) -> BypassRelay
- R35 pad 1: Net-(Q1-G) -> Net-(Q5-G)
- R36 pad 1: Net-(Q2-G) -> Net-(Q6-G)
- R46 pad 1: CTout -> CTOut
- R51 pad 1: ZCDA -> Net-(U15-+)
- R52 pad 1: ZCDB -> Net-(U15--)
- R7 pad 1: GND -> Net-(LED1-Pad2)
- R7 pad 2: Net-(J1-SHIELD) -> D3.3V
- U2 pad 1: 24V -> GND
- U2 pad 2: 24V -> Net-(U2-SW)
- U2 pad 3: Net-(U2-LX) -> 24V
- U2 pad 5: GND -> 24V
- U3 pad 1: Net-(J3-Pin_2) -> 5V
- U3 pad 3: Net-(J3-Pin_1) -> 5V
- U3 pad 4: Net-(R12-Pad1) -> Net-(U3-FB)
- U3 pad 5: 3.3V -> A3.6V
- U8 pad 12: IO8 -> DAC_CLK
- U8 pad 15: ZCDA -> IO3
- U8 pad 17: IO9 -> DAC_DOUT
- U8 pad 18: IO10 -> ADC_CS
- U8 pad 19: PrimaryRelay -> ADC_DIN
- U8 pad 2: 3.3V -> D3.3V
- U8 pad 20: BypassRelay -> ADC_CLK
- U8 pad 21: GD1-A -> ADC_DOUT
- U8 pad 23: IO21 -> OCDInterrupt
- U8 pad 24: IO47 -> LED4
- U8 pad 25: IO48 -> ZCDInterrupt
- U8 pad 26: IO45 -> LED3
- U8 pad 31: IO38 -> GD1-A
- U8 pad 32: IO39 -> BypassRelay
- U8 pad 33: IO40 -> PrimaryRelay
- U8 pad 34: IO41 -> LED1
- U8 pad 35: IO42 -> LED2
- U8 pad 38: CTout -> IO2
- U8 pad 39: VBUS -> IO1
- U8 pad 4: ZCDB -> IO4
- U8 pad 5: Therm1 -> IO5
- U8 pad 6: Therm2 -> DAC_CS
- U8 pad 7: IO7 -> DAC_DIN
Routing:
- net A3.6V: track 0.00 -> 408.0 mm, vias 0 -> 10
- net D3.3V: track 0.00 -> 218.8 mm, vias 0 -> 7
- net 24V: track 85.3 -> 248.1 mm, vias 9 -> 18
- net ZCDB: track 65.0 -> 0.00 mm, vias 2 -> 0
- net ZCDInterrupt: track 0.00 -> 57.3 mm, vias 0 -> 2
- net CTout: track 54.8 -> 0.00 mm, vias 2 -> 0
- net OCDInterrupt: track 0.00 -> 53.3 mm, vias 0 -> 4
- net LED1: track 0.00 -> 48.1 mm, vias 0 -> 2
- net GND: track 120.7 -> 168.7 mm, vias 60 -> 118
- net ZCDA: track 46.5 -> 0.00 mm, vias 2 -> 0
- net LED2: track 0.00 -> 45.4 mm, vias 0 -> 2
- net LED4: track 0.00 -> 40.4 mm, vias 0 -> 2
- net DAC_CS: track 0.00 -> 40.2 mm, vias 0 -> 2
- net LED3: track 0.00 -> 38.0 mm
- net DAC_DIN: track 0.00 -> 36.3 mm, vias 0 -> 2
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- added copper zone on B.Cu, net 24V
- added copper zone on F.Cu, net 24V
- added copper zone on F.Cu, net GND
- added copper zone on In2.Cu, net GND
- added copper zone on B.Cu, net Net-(U2-SW)
- added copper zone on F.Cu, net Net-(U2-SW)
- removed copper zone on In2.Cu, net 24V
- removed copper zone on In2.Cu, net 3.3V
- removed copper zone on In2.Cu, net 5V
Other:
- board text added: "12/3/2025 (MDY)"
- board text added: "24V"
- board text added: "5V"
- board text added: "A3.6V"
- board text added: "Analog In"
- board text added: "D3.3V"
- board text added: "IO1"
- board text added: "IO2"
- board text added: "IO3"
- board text added: "IO4"
- board text added: "IO5"
- board text added: "Musical DRSSTC Rev 2.0"
- board text removed: "+3.3V"
- board text removed: "+5V"
- board text removed: "8/11/2025 (MDY)"
- board text removed: "IO10"
- board text removed: "IO15"
- board text removed: "IO21"
- board text removed: "IO38"
- board text removed: "IO39"
- board text removed: "IO40"
- board text removed: "IO41"
- board text removed: "IO42"
- board text removed: "IO45"
- board text removed: "IO47"
- board text removed: "IO48"
- board text removed: "IO7"
- board text removed: "IO8"
- board text removed: "IO9"
- board text removed: "Musical DRSSTC Rev 1.0"
