File: KiCad-9/MusicalTeslaCoil.kicad_sch (KiCad schematic)
At the start: 116 parts, among them J1 USB_C-UJ20-C-H-C-MSMT-TR, J10 NTC Thermistor 2, J11 Conn_01x10_Pin, J12 Conn_01x05_Pin, J13 Conn_01x06_Pin, J14 Conn_02x03_Odd_Even, J2 Power in, J3 VBUS, J4 Primary Relay, J5 Soft Start Bypass Relay, J6 Current Transformer, J7 GDT1, J8 GDT2, J9 NTC Thermistor 1, Q1 PMV20ENR, Q2 PMV20ENR, SW1 USB Boot, SW2 Reset, U1 ESP32-S3-WROOM-1, U10 AP2112K-3.3TRG1, U2 R1240N001B-TR-FE, U3 LMV321, U4 DMC4029SK4-13, U5 UCC27423DR, U6 DMC4029SK4-13, U7 UCC27423DR, U8 DMC4029SK4-13, U9 DMC4029SK4-13

Commit message: Uploaded Rev 2.0
Parts:
- removed C36, C37: 0.1uF, Capacitor_SMD:C_0805_2012Metric_Pad1.18x1.45mm_HandSolder, symbol Device:C
- removed C38, C39: 1uF, Capacitor_SMD:C_0805_2012Metric_Pad1.18x1.45mm_HandSolder, symbol Device:C
- removed C40: 10uF, Capacitor_SMD:C_0805_2012Metric_Pad1.18x1.45mm_HandSolder, symbol Device:C
- removed C41: 470pF, Capacitor_SMD:C_0805_2012Metric_Pad1.18x1.45mm_HandSolder, symbol Device:C
- removed CR12: MSS1P4-M3/89A, DIODE_MSP3V3, symbol MSS1P4_M3_89A:MSS1P4-M3_89A
- removed CR13: CMS06TE12L_Q_M, M-FLAT_TOS, symbol CMS06_TE12L_Q_M_:CMS06TE12L_Q_M
- removed J1: USB_C-UJ20-C-H-C-MSMT-TR, Connector_USB:USB_C-UJ20-C-H-C-MSMT-TR, symbol UJ20-C-H-C-MSMT-TR:USB_C-UJ20-C-H-C-MSMT-TR
- removed J11: Conn_01x10_Pin, Connector_PinHeader_2.54mm:PinHeader_1x10_P2.54mm_Vertical, symbol Connector:Conn_01x10_Pin
- removed J12: Conn_01x05_Pin, Connector_PinHeader_2.54mm:PinHeader_1x05_P2.54mm_Vertical, symbol Connector:Conn_01x05_Pin
- removed J13: Conn_01x06_Pin, Connector_PinHeader_2.54mm:PinHeader_1x06_P2.54mm_Vertical, symbol Connector:Conn_01x06_Pin
- removed J14: Conn_02x03_Odd_Even, Connector_PinHeader_2.54mm:PinHeader_2x03_P2.54mm_Vertical, symbol Connector_Generic:Conn_02x03_Odd_Even
- removed L1: SLF7045T-4R7M2R0-PF, IND_7045_TDK, symbol SLF7045T_4R7M2R0_PF:SLF7045T-4R7M2R0-PF
- removed Q1, Q2: PMV20ENR, PMV20ENR:QNMOS1G2S3D_TO-236AB_SOT23_NEX, symbol PMV20ENR:PMV20ENR
- removed R34: 51, Resistor_SMD:R_0805_2012Metric_Pad1.20x1.40mm_HandSolder, symbol Device:R_US
- removed R35: 6.3k 1%, Resistor_SMD:R_0805_2012Metric_Pad1.20x1.40mm_HandSolder, symbol Device:R_US
- removed R36: 1.2k 1%, Resistor_SMD:R_0805_2012Metric_Pad1.20x1.40mm_HandSolder, symbol Device:R_US
- removed U10: AP2112K-3.3TRG1, AP2112K_3_3TRG1:SOT95P285X140-5N, symbol AP2112K-3.3TRG1:AP2112K-3.3TRG1
- removed U2: R1240N001B-TR-FE, SOT-23-6W_PE-SOT23-6W-0512_NMD, symbol R1240N001B_TR_FE:R1240N001B-TR-FE
- removed U3: LMV321, footprints:DCK5_TEX, symbol Amplifier_Operational:LMV321
- added C13, C15, C16, C4: 10nF, Capacitor_SMD:C_0805_2012Metric_Pad1.18x1.45mm_HandSolder, symbol Device:C
- added C14: 0.1uF, Capacitor_SMD:C_0805_2012Metric_Pad1.18x1.45mm_HandSolder, symbol Device:C
- added C17, C19, C2: 10uF, Capacitor_SMD:C_0805_2012Metric_Pad1.18x1.45mm_HandSolder, symbol Device:C
- added C18, C20, C22, C29, C3: 2.2uF, Capacitor_SMD:C_0805_2012Metric_Pad1.18x1.45mm_HandSolder, symbol Device:C
- added C21: 1nF, Capacitor_SMD:C_0805_2012Metric_Pad1.18x1.45mm_HandSolder, symbol Device:C
- added C45, C46, C6: 1uF, Capacitor_SMD:C_0805_2012Metric_Pad1.18x1.45mm_HandSolder, symbol Device:C
- added C53: 470pF, Capacitor_SMD:C_0805_2012Metric_Pad1.18x1.45mm_HandSolder, symbol Device:C
- added CR1, CR10, CR9: MSS1P4-M3/89A, DIODE_MSP3V3, symbol MSS1P4_M3_89A:MSS1P4-M3_89A
- added D9: BZT52C15-7-F, Diode_SMD:D_SOD-123, symbol Device:D_Zener
- added F1: 0ZCG0050AF2C, 0ZCG0050AF2C:FUSER_0ZCG0050AF2C, symbol 0ZCG0050AF2C:0ZCG0050AF2C
- added H1, H2, H3, H4: MountingHole, MountingHole:MountingHole_3.2mm_M3, symbol Mechanical:MountingHole
- added J11, J12, J13, J14: Conn_01x02, Connector_Molex:Molex_KK-254_AE-6410-02A_1x02_P2.54mm_Vertical, symbol Connector_Generic:Conn_01x02
- added J17: Conn_01x05, Connector_PinHeader_2.54mm:PinHeader_1x05_P2.54mm_Vertical, symbol Connector_Generic:Conn_01x05
- added J18: Conn_01x07, Connector_PinHeader_2.54mm:PinHeader_1x07_P2.54mm_Vertical, symbol Connector_Generic:Conn_01x07
- added J2: Conn_01x03, Connector_Molex:Molex_KK-254_AE-6410-03A_1x03_P2.54mm_Vertical, symbol Connector_Generic:Conn_01x03
- added J3: USB4215-03-A, USB4215_03_A:USB4215_03_A, symbol USB4215_03_A:USB4215-03-A_REVA
- added L1: VLS6045EX-150M, VLS6045EX_150M:VLS6045EX_150M, symbol VLS6045EX-150M:VLS6045EX-150M
- added LED1, LED5: LTST-C170GKT, LTST_C170GKT:LED_LTST-C170GKT_LTO, symbol LTST_C170GKT:LTST-C170GKT
- added LED2: LTST-C170KFKT, LTST_C170KFKT:LED_LTST-C170KFKT_LTO, symbol LTST_C170KFKT:LTST-C170KFKT
- added LED3: LTST-C171KRKT, LTST_C171KRKT:LED_LTST-C171_LTO, symbol LTST_C171KRKT:LTST-C171KRKT
- added LED4: LTST-C170KSKT, LTST_C170KSKT:LED_LTST-C170KSKT_LTO, symbol LTST_C170KSKT:LTST-C170KSKT
- added Q1: GSF3407, Package_TO_SOT_SMD:SOT-23, symbol Transistor_FET:Q_PMOS_GSD
- added Q2: SSF7912, Package_TO_SOT_SMD:SOT-23, symbol SSF7912:SSF7912
- added Q5, Q6: 2N7002K, Package_TO_SOT_SMD:SOT-23, symbol SSF7912:SSF7912
- added R1, R18, R6: 5.1k, Resistor_SMD:R_0805_2012Metric_Pad1.20x1.40mm_HandSolder, symbol Device:R_US
- added R10: 100k, Resistor_SMD:R_0805_2012Metric_Pad1.20x1.40mm_HandSolder, symbol Device:R_US
- added R12, R17: 1k, Resistor_SMD:R_0805_2012Metric_Pad1.20x1.40mm_HandSolder, symbol Device:R_US
- added R14, R15, R21, R22, R57: 150, Resistor_SMD:R_0805_2012Metric_Pad1.20x1.40mm_HandSolder, symbol Device:R_US
- added R16: 0, Resistor_SMD:R_0805_2012Metric_Pad1.20x1.40mm_HandSolder, symbol Device:R_US
- added R19, R2, R24, R29: 3k, Resistor_SMD:R_0805_2012Metric_Pad1.20x1.40mm_HandSolder, symbol Device:R_US
- added R20: 16.5k, Resistor_SMD:R_0805_2012Metric_Pad1.20x1.40mm_HandSolder, symbol Device:R_US
- added R23: 22k, Resistor_SMD:R_0805_2012Metric_Pad1.20x1.40mm_HandSolder, symbol Device:R_US
- added R25: 10k, Resistor_SMD:R_0805_2012Metric_Pad1.20x1.40mm_HandSolder, symbol Device:R_US
- added R26: 51, Resistor_SMD:R_0805_2012Metric_Pad1.20x1.40mm_HandSolder, symbol Device:R_US
- added R58: 200k, Resistor_SMD:R_0805_2012Metric_Pad1.20x1.40mm_HandSolder, symbol Device:R_US
- added U1, U3: TLV75801PDBV, Package_TO_SOT_SMD:SOT-23-5, symbol Regulator_Linear:TLV75801PDBV
- added U15, U16: NCS2250SQ2T2G, NCS2250SQ2T2G:SC70-5_2P2X1P35_ONS, symbol NCS2250SQ2T2G:NCS2250SQ2T2G
- added U2: TPP362082-T6TR, TPP362082_T6TR:TSOT23-6-A_TPK, symbol TPP362082_T6TR:TPP362082-T6TR
- added U4: MCP3204T-CI/SL, MCP3204T_CI_SL:SOIC14-N_MC_MCH, symbol MCP3204T_CI_SL:MCP3204T-CI_SL
- added U5: MCP48FVB11, MCP48FVB11:MCP48FVB11, symbol MCP48FVB11:MCP48FVB11
- added U6: MCP1501T-33E/CHY, MCP1501T_33E_CHY:SOT-23-6_CHY_MCH, symbol MCP1501T_33E_CHY:MCP1501T-33E_CHY
- added U7: MCP6006UT-E/LT, MCP6006UT_E_LT:SC70-5_LT_MCH, symbol MCP6006UT_E_LT:MCP6006UT-E_LT
- C1: value 0.1uF -> 2.2uF
- C26: renamed from C42; value 1uF -> 0.1uF
- C5: value 10uF -> 2.2uF
- C7: value 1nF -> 10nF
- CR11: renamed from CR8; value 1N4007FL -> 1N4148WS-7-F; footprint CR_SOD-123FL_SME -> 1N4148WX_TP:CR_SOD323_MCC
- CR12: renamed from CR9; value 1N4007FL -> 1N4148WS-7-F; footprint CR_SOD-123FL_SME -> 1N4148WX_TP:CR_SOD323_MCC
- CR13: renamed from CR10; value 1N4007FL -> 1N4148WS-7-F; footprint CR_SOD-123FL_SME -> 1N4148WX_TP:CR_SOD323_MCC
- CR14: renamed from CR11; value 1N4007FL -> 1N4148WS-7-F; footprint CR_SOD-123FL_SME -> 1N4148WX_TP:CR_SOD323_MCC
- CR2: renamed from CR1; footprint CR_SOD-123FL_SME -> 1N4007FL:CR_SOD-123FL_SME
- CR3: renamed from CR2; footprint CR_SOD-123FL_SME -> 1N4007FL:CR_SOD-123FL_SME
- CR5: renamed from CR4; footprint DO-214AA_VIS -> ES2B_E3_52T:DO-214AA_VIS
- CR6: renamed from CR3; footprint DO-214AA_VIS -> ES2B_E3_52T:DO-214AA_VIS
- CR7: renamed from CR6; footprint DO-214AA_VIS -> ES2B_E3_52T:DO-214AA_VIS
- CR8: renamed from CR5; footprint DO-214AA_VIS -> ES2B_E3_52T:DO-214AA_VIS
- R11: value 5.1k -> 1k
- R27: renamed from R10; value 3k 1% -> 1.5k
- R3: value 5.1k -> 15k
- R31: renamed from R12; value 3k 1% -> 3k
- R33: renamed from R14; value 1k -> 10k
- R34: renamed from R17; value 1k -> 10k
- R37: renamed from R32; value 1k 1% -> 1k
- R38: renamed from R33; value 1k 1% -> 1k
- R51: renamed from R18; value 100 -> 1k
- R52: renamed from R19; value 100 -> 1k
- R7: value 100k -> 150
- renumbered C6 to C23, C4 to C24, C2 to C25, C43 to C27, C3 to C28, C14 to C30, C15 to C31, C13 to C32, C17 to C33, C18 to C34, C27 to C35, C16 to C36, C19 to C37, C24 to C38, C28 to C39, C29 to C40, C20 to C41, C25 to C42, C30 to C43, C31 to C44, C21 to C47, C26 to C48, C32 to C49, C33 to C50, C22 to C51, C34 to C52, C23 to C54, C35 to C55, CR7 to CR4, J2 to J1, J5 to J10, J7 to J15, J8 to J16, J3 to J4, J6 to J5, J9 to J6, J10 to J7, J4 to J9, R6 to R28, R1 to R30, R2 to R32, R15 to R35, R16 to R36, R23 to R39, R27 to R43, R22 to R44, R28 to R45, R21 to R46, R20 to R47, R38 to R48, R37 to R49, R39 to R50, R24 to R53, R26 to R54, R29 to R55, R30 to R56, R25 to R59, R31 to R60, U7 to U10, U4 to U11, U6 to U12, U8 to U13, U9 to U14, U1 to U8, U5 to U9
Connections:
- net IO38 is gone; now on net GD1-A: U8.31 (IO38)
- net IO39 is gone; now on net BypassRelay: U8.32 (IO39)
- net IO40 is gone; now on net PrimaryRelay: U8.33 (IO40)
- net 24V: now also C2.1, F1.1, J11.1 (Pin_1), Q2.1 (G), R25.2, U2.3 (VIN), U2.5 (EN); no longer C5.1, J1.2 (Pin_2)
- net 5V: now also C1.2, C5.2, CR1.1, J12.1 (Pin_1), Q2.3 (D), U1.1 (IN), U1.3 (EN), U3.1 (IN), U3.3 (EN)
- net BypassRelay: now also R34.1; no longer U8.20 (IO12)
- net GD1-A: no longer U8.21 (IO13)
- net GND: now also C1.1, C5.1, C13.1, C15.1, C17.2, C18.1, C19.2, C2.2, C20.1, C21.1, C22.1, C29.1, C3.1, C4.1, C45.1, C46.1, C6.1, CR10.2, CR9.2, J11.2 (Pin_2), J12.2 (Pin_2), J13.2 (Pin_2), J14.2 (Pin_2), J2.1 (Pin_1), J3.A1_B12 (GND_A), J3.B1_A12 (GND_B), LED1.1, LED2.1, LED3.1, LED4.1, LED5.1, Q5.2 (S), Q6.2 (S), R1.1, R10.2, R18.1, R20.1, R24.1, R25.1, R29.1, R6.1, U1.2 (GND), U15.2 (V-), U16.2 (V-), U2.1 (GND), U3.2 (GND), U4.12 (AGND), U4.7 (DGND), U5.7 (GND), U6.2 (GND), U6.3 (GND), U6.5 (GND), U7.2 (V-); no longer C5.2, R11.1, R7.1
- net IO17: now also J17.3 (Pin_3)
- net IO18: now also J17.4 (Pin_4)
- net IO35: now also J18.7 (Pin_7)
- net IO36: now also J18.6 (Pin_6)
- net IO37: now also J18.5 (Pin_5)
- net PrimaryRelay: now also R33.1; no longer U8.19 (IO11)
- net RXD0: now also J18.4 (Pin_4)
- net TXD0: now also J18.3 (Pin_3)
- net Therm1: now also R13.2; no longer U8.5 (IO5)
- net Therm2: now also R12.2; no longer U8.6 (IO6)
- net USB_D+: now also J3.A6 (DP1), J3.B6 (DP2)
- net USB_D-: now also J3.A7 (DN1), J3.B7 (DN2)
- net VBUS: now also R31.1, R17.2, U7.4; no longer C7.2, R13.1, U8.39 (IO1)
- net at J4.1 (Pin_1), R31.2: now also R29.2, U7.3 (-)
- net at R3.2: now also R2.1, U1.4 (FB)
- net at R36.1: now also Q6.1 (G); no longer R34.1
- net D3.3V: now reaches R7.2
- net D3.3V: now also C27.2, C28.1, R28.1, R30.1, U8.2 (3V3), C3.2, J14.1 (Pin_1), R2.2, U1.5 (OUT)
- net at C23.2, J4.2 (Pin_2), R27.2: now also U7.1 (+)
- net at CR2.2, J9.2 (Pin_2): now also Q5.3 (D)
- net at CR3.2, J10.2 (Pin_2): now also Q6.3 (D)
- net at R35.1: now also Q5.1 (G); no longer R33.1
- net at R11.2: now also J2.3 (Pin_3)
- removed net 3.3V: C26.2, C27.2, C28.1, J6.2 (Pin_2), J7.2 (Pin_2), R28.1, R30.1, U8.2 (3V3)
- net CTout renamed CTOut
- net CTOut: now also R57.2, R58.2, U16.3 (+); no longer U8.38 (IO2)
- net IO10 renamed ADC_CS
- net ADC_CS: now also U4.8 (*CS/SHDN)
- net IO21 renamed OCDInterrupt
- net OCDInterrupt: now also C53.1, R58.1, U16.1
- net IO41 renamed LED1
- net LED1: now also R15.2
- net IO42 renamed LED2
- net LED2: now also R22.2
- net IO45 renamed LED3
- net LED3: now also R14.2
- net IO47 renamed LED4
- net LED4: now also R21.2
- net IO48 renamed ZCDInterrupt
- net ZCDInterrupt: now also U15.1
- net IO7 renamed DAC_DIN
- net DAC_DIN: now also U5.10 (SDI)
- net IO8 renamed DAC_CLK
- net DAC_CLK: now also U5.9 (SCK)
- net IO9 renamed DAC_DOUT
- net DAC_DOUT: now also U5.8 (SDO)
- net ZCDA: no longer names the net of C36.2, R51.1
- net ZCDA: now also CR9.1, U15.3 (+); no longer U8.15 (IO3)
- net ZCDB: no longer names the net of C36.1, R52.1
- net ZCDB: now also CR10.1, U15.4 (-); no longer U8.4 (IO4)
- new net: C13.2, R13.1, U4.2 (CH1)
- new net: C15.2, R17.1, U4.1 (CH0)
- new net: LED4.2, R21.1
- new net: CR1.2, J3.A4_B9 (VBUS_A), J3.B4_A9 (VBUS_B)
- new net: J3.A5 (CC1), R6.2
- new net: J3.B5 (CC2), R18.2
- new net: J3.SH4 (SHIELD__3), R10.1
- new net: L1.1, R16.2, U2.2 (SW)
- new net: R23.1, R24.2, U2.4 (VFB)
- new net: C14.1, U2.6 (VBST)
- new net: C16.1, R19.1, R20.2, U3.4 (FB)
- new net: LED1.2, R7.1
- new net: C7.2, R12.1, U4.3 (CH2)
- new net: LED2.2, R14.1
- new net: D9.1 (K), F1.2, Q1.2 (S)
- new net: C21.2, R26.2, U4.13 (VREF), U6.1 (OUT)
- new net: C53.2, R57.1
- new net: C17.1, C19.1, L1.2, Q2.2 (S), R23.2
- new net: C14.2, R16.1
- new net: C4.2, R11.1, U4.4 (CH3)
- new net: LED3.2, R15.1
- new net: LED5.2, R22.1
- new net: D9.2 (A), Q1.1 (G), R1.2
- new net: C22.2, R26.1
- new net: J1.2 (Pin_2), Q1.3 (D)
- new net A3.6V: C16.2, C18.2, C20.2, C26.2, C29.2, C45.2, C46.2, C6.2, J13.1 (Pin_1), J2.2 (Pin_2), J6.2 (Pin_2), J7.2 (Pin_2), R19.2, U15.5 (V+), U16.5 (V+), U3.5 (OUT), U4.14 (VDD), U5.1 (VDD), U6.4 (*SHDN), U6.6 (VDD), U7.5 (V+)
- new net ADC_CLK: U4.11 (CLK), U8.20 (IO12)
- new net ADC_DIN: U4.9 (DIN), U8.19 (IO11)
- new net ADC_DOUT: U4.10 (DOUT), U8.21 (IO13)
- new net DACVOut: U16.4 (-), U5.4 (VOut)
- new net DAC_CS: U5.2 (*CS), U8.6 (IO6)
- new net IO1: J18.1 (Pin_1), U8.39 (IO1)
- new net IO2: J18.2 (Pin_2), U8.38 (IO2)
- new net IO3: J17.5 (Pin_5), U8.15 (IO3)
- new net IO4: J17.1 (Pin_1), U8.4 (IO4)
- new net IO5: J17.2 (Pin_2), U8.5 (IO5)
- no-connect marks 2 -> 4
Other:
- note added: "ADC"
- note added: "Add a 1k 10nF RC filter for each ADC input in use"
- note added: "Add a power on LED, and add 4 LED's connected to GPIO"
- note added: "Add another LDO for A3.6v rail, make sure LDO's PSRR is sufficient for the switching regulators frequency"
- note added: "Add comparator and peak detector circuit to CT circuit"
- note added: "Add mounting holes"
- note added: "Add protection circuitry: Reverse polarity, over current"
- note added: "Completed:"
- note added: "DAC"
- note added: "Edit IC symbols to be their actual component symbols"
- note added: "Isolated primary current measurement for measurement and ZCS"
- note added: "LED's"
- note added: "Make GDT2 pcb layout the same as GDT1"
- note added: "Make sure USB-C footprint is correct"
- note added: "Make sure feedback resistors are atleast 0.5% tolerance"
- note added: "Mounting Holes"
- note added: "OCD circuit with comparator and DAC"
- note added: "PCB Specific:"
- note added: "Power in = 24V"
- note added: "Redo PCB stackup to SIG/POWER - GND - GND - SIG/POWER"
- note added: "Replace GDT diodes with a fast recovery diode"
- note added: "Revision Todos:"
- note added: "Use a cheaper buck regulator"
- note added: "Use molex 2.54mm connectors instead of dupont connectors"
- note added: "^^^ Reverse protection against USB power"
- note added: "add a decent external ADC"
- note removed: "Isolated primary current measurement for data and ZCS"
- moved on the sheet: C30, C31, C32, C33, C36, CR4, CR5, CR6, CR7, CR8, FL1, J1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
