File: KiCad-9/PrimaryCircuit.kicad_sch (KiCad schematic)
At the start: 26 parts, among them K1 Relay_SPST-NO, K2 Relay_SPST-NO, Q3 SKM100GB125DN, Q4 SKM100GB125DN

Commit message: Uploaded Rev 2.0
Parts:
- C11, C12: value 6000uF 350V -> 3000uF 400V
Changed lines of the file:
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@@
 			)
 		)
-		(property "Value" "6000uF 350V"
+		(property "Value" "3000uF 400V"
 			(at 140.97 128.524 0)
 			(effects
@@
 			)
 		)
-		(property "Description" "Polarized capacitor, SIEMENS B43471"
+		(property "Description" "Polarized capacitor, KEMET ALS70A302KF400"
 			(at 146.05 120.65 0)
 			(effects
@@
 			)
 		)
-		(property "Value" "6000uF 350V"
+		(property "Value" "3000uF 400V"
 			(at 139.7 84.074 0)
 			(effects
@@
 			)
 		)
-		(property "Description" "Polarized capacitor, SIEMENS B43471"
+		(property "Description" "Polarized capacitor, KEMET ALS70A302KF400"
 			(at 146.05 90.17 0)
 			(effects
